Commit message: added shin sensor

File: urdfs/leg/leg.gazebo.xacro (robot description, xacro)
@@ -58,4 +58,14 @@
 			<maxVel>1.0</maxVel>
 			<minDepth>0.00</minDepth>
+			<sensor name="${name}_shin_contact_sensor" type="contact">
+                <always_on>true</always_on>
+                <update_rate>1000.0</update_rate>
+                <contact>
+                  <collision>${name}_lowerleg_collision</collision>
+                </contact>
+                <plugin name="${name}_shin_bumper" filename="libgazebo_ros_bumper.so">
+                  <bumperTopicName>/${name}_shin_sensor</bumperTopicName>
+                </plugin>
+            </sensor>
 		</gazebo>
 		<gazebo reference="${name}_foot">
