Commit message: using cylidners for legcollision in lowerleg

File: urdfs/leg/leg.urdf.xacro (robot description, xacro)
@@ -113,6 +113,7 @@
 			</visual>
 			<collision>
+			    <origin xyz="${lowerleg_length/2.0} 0 0" rpy="0 ${-PI/2}  0"/>
 				<geometry>
-					<mesh filename="package://hyq_description/meshes/leg/lowerleg.dae" scale="1 1 1"/>
+					<cylinder length="${lowerleg_length}"  radius="0.02"/>
 				</geometry>
 			</collision>

Commit message: [bugfix] wrong variable to set kin limits

File: urdfs/leg/leg.urdf.xacro (robot description, xacro)
@@ -14,5 +14,5 @@
 			<child  link="${name}_hipassembly"/>
 			<axis xyz="0 0 1"/>
-			<limit effort="${haa_limit}" velocity="12.0" lower="${haa_min*PI/180}" soft_upper_limit="${haa_max*PI/180}" />
+			<limit effort="${haa_limit}" velocity="12.0" lower="${haa_min*PI/180}" upper="${haa_max*PI/180}" />
 			<dynamics damping="0.1" friction="0" />
 			<safety_controller k_position="50" k_velocity="10"
@@ -30,6 +30,6 @@
 			<dynamics damping="0.1" friction="0" />
 			<safety_controller k_position="50" k_velocity="10"
-                  lower="${(1-knee_bent_backward)*(hfe_min)*PI/180 + (knee_bent_backward)*(-hfe_max)*PI/180}"
-                  upper="${(1-knee_bent_backward)*(hfe_max)*PI/180 + (knee_bent_backward)*(-hfe_min)*PI/180}"/>
+                  soft_lower_limit="${(1-knee_bent_backward)*(hfe_min)*PI/180 + (knee_bent_backward)*(-hfe_max)*PI/180}"
+                  soft_upper_limit="${(1-knee_bent_backward)*(hfe_max)*PI/180 + (knee_bent_backward)*(-hfe_min)*PI/180}"/>
 		</joint>
 		<!-- Lower leg joint -->
@@ -44,6 +44,6 @@
 			<dynamics damping="0.1" friction="0" />
 			<safety_controller k_position="50" k_velocity="10"
-                  lower="${(1-knee_bent_backward)*(kfe_min)*PI/180 + (knee_bent_backward)*(-kfe_max)*PI/180}"
-                  upper="${(1-knee_bent_backward)*(kfe_max)*PI/180 + (knee_bent_backward)*(-kfe_min)*PI/180}"/>
+                  soft_lower_limit="${(1-knee_bent_backward)*(kfe_min)*PI/180 + (knee_bent_backward)*(-kfe_max)*PI/180}"
+                  soft_upper_limit="${(1-knee_bent_backward)*(kfe_max)*PI/180 + (knee_bent_backward)*(-kfe_min)*PI/180}"/>
 		<!-- Foot joint -->
 		</joint>
