Commit message: added knee_kent_backwards, lowerleg_length, upperleg_length to be consistent with hyqreal
added also possibility to set torque limits and kinematic limits from
commons.xacro

File: robots/hyq.urdf.xacro (robot description, xacro)
@@ -44,4 +44,5 @@
 		reflect_upper="1"
 		reflect_front="1"
+		knee_bent_backward="1"
 		load_force_sensors="$(arg load_force_sensors)">
 		<origin xyz="${d_fh/2} ${d_lr/2} 0" rpy="0 ${PI/2} ${PI}"/>
@@ -54,4 +55,5 @@
 		reflect_upper="-1"
 		reflect_front="1"
+		knee_bent_backward="1"
 		load_force_sensors="$(arg load_force_sensors)">
 		<origin xyz="${d_fh/2} ${-d_lr/2} 0" rpy="0 ${PI/2} 0"/>
@@ -64,4 +66,5 @@
 		reflect_upper="1"
 		reflect_front="-1"
+		knee_bent_backward="0"
 		load_force_sensors="$(arg load_force_sensors)">
 		<origin xyz="${-d_fh/2} ${d_lr/2} 0" rpy="0 ${PI/2} ${PI}"/>
@@ -74,4 +77,5 @@
 		reflect_upper="-1"
 		reflect_front="-1"
+		knee_bent_backward="0"
 		load_force_sensors="$(arg load_force_sensors)">
 		<origin xyz="${-d_fh/2} ${-d_lr/2} 0" rpy="0 ${PI/2} 0"/>

File: robots/hyq_model.urdf.xacro (robot description, xacro)
@@ -29,4 +29,5 @@
 		reflect_upper="1"
 		reflect_front="1"
+		knee_bent_backward="1"
 		load_force_sensors="false">
 		<origin xyz="${d_fh/2} ${d_lr/2} 0" rpy="0 ${PI/2} ${PI}"/>
@@ -39,4 +40,5 @@
 		reflect_upper="-1"
 		reflect_front="1"
+		knee_bent_backward="1"
 		load_force_sensors="false">
 		<origin xyz="${d_fh/2} ${-d_lr/2} 0" rpy="0 ${PI/2} 0"/>
@@ -49,4 +51,5 @@
 		reflect_upper="1"
 		reflect_front="-1"
+		knee_bent_backward="0"
 		load_force_sensors="false">
 		<origin xyz="${-d_fh/2} ${d_lr/2} 0" rpy="0 ${PI/2} ${PI}"/>
@@ -59,4 +62,5 @@
 		reflect_upper="-1"
 		reflect_front="-1"
+		knee_bent_backward="0"
 		load_force_sensors="false">
 		<origin xyz="${-d_fh/2} ${-d_lr/2} 0" rpy="0 ${PI/2} 0"/>

File: robots/hyq_no_sensors.urdf.xacro (robot description, xacro)
@@ -34,4 +34,5 @@
 		reflect_upper="1"
 		reflect_front="1"
+		knee_bent_backward="1"
 		load_force_sensors="$(arg load_force_sensors)">
 		<origin xyz="${d_fh/2} ${d_lr/2} 0" rpy="0 ${PI/2} ${PI}"/>
@@ -44,4 +45,5 @@
 		reflect_upper="-1"
 		reflect_front="1"
+		knee_bent_backward ="1"
 		load_force_sensors="$(arg load_force_sensors)">
 		<origin xyz="${d_fh/2} ${-d_lr/2} 0" rpy="0 ${PI/2} 0"/>
@@ -54,4 +56,5 @@
 		reflect_upper="1"
 		reflect_front="-1"
+		knee_bent_backward="0"
 		load_force_sensors="$(arg load_force_sensors)">
 		<origin xyz="${-d_fh/2} ${d_lr/2} 0" rpy="0 ${PI/2} ${PI}"/>
@@ -64,4 +67,5 @@
 		reflect_upper="-1"
 		reflect_front="-1"
+		knee_bent_backward="0"
 		load_force_sensors="$(arg load_force_sensors)">
 		<origin xyz="${-d_fh/2} ${-d_lr/2} 0" rpy="0 ${PI/2} 0"/>

File: urdfs/common.xacro (robot description, xacro)
@@ -2,10 +2,21 @@
 <robot>
 	<property name="PI" value="3.1415926535897931"/>
+    <!-- kin limits (sign ref is RH leg)-->
+    <property name="haa_max" value="25"/>
+    <property name="haa_min" value="-70"/>
+    <property name="hfe_max" value="50"/>
+    <property name="hfe_min" value="-70"/>
+    <property name="kfe_max" value="140"/>
+    <property name="kfe_min" value="20"/>
+    <!-- torque limits 120-->
+    <property name="haa_limit" value="150"/>
+    <property name="hfe_limit" value="150"/>
+    <property name="kfe_limit" value="150"/>
 	<!-- standard distances -->
 	<property name="d_lr" value="0.414"/>
 	<property name="d_fh" value="0.747"/>
-	<property name="d_p0p1" value="0.08"/>
-	<property name="d_p1p2" value="0.35"/>
-	<property name="d_p2p3" value="0.346"/>
+	<property name="hipassembly_length" value="0.08"/>
+	<property name="upperleg_length" value="0.35"/>
+	<property name="lowerleg_length" value="0.346"/>
 	<!-- Inertial values -->
 	<!-- Trunk with hydraulic system -->

File: urdfs/leg/leg.urdf.xacro (robot description, xacro)
@@ -6,5 +6,5 @@
 	<!-- ================================== Leg ================================== -->
 	<!-- The xacro macro xacro:hyq_leg contains: hip assembly, upper and lower leg -->
-	<xacro:macro name="hyq_leg" params="name parent *origin reflect_hip reflect_upper reflect_front load_force_sensors">
+	<xacro:macro name="hyq_leg" params="name parent *origin reflect_hip reflect_upper reflect_front knee_bent_backward load_force_sensors">
 		<!-- Joints -->
 		<!-- Hip assembly joint -->
@@ -14,40 +14,40 @@
 			<child  link="${name}_hipassembly"/>
 			<axis xyz="0 0 1"/>
-			<limit effort="150.0" velocity="12.0" lower="${-7*PI/18}" upper="${5*PI/36}"/>
+			<limit effort="${haa_limit}" velocity="12.0" lower="${haa_min*PI/180}" soft_upper_limit="${haa_max*PI/180}" />
 			<dynamics damping="0.1" friction="0" />
-			<safety_controller k_position="100" k_velocity="100"
-							   soft_lower_limit="${-7*PI/18}" soft_upper_limit="${5*PI/36}" />
+			<safety_controller k_position="50" k_velocity="10"
+							   soft_lower_limit="${haa_min*PI/180}" soft_upper_limit="${haa_max*PI/180}" />
 		</joint>
 		<!-- Upper leg joint -->
 		<joint name="${name}_hfe_joint" type="revolute">
-			<origin xyz="${d_p0p1} 0 0" rpy="${reflect_upper*PI/2} 0 0"/>
+			<origin xyz="${hipassembly_length} 0 0" rpy="${reflect_upper*PI/2} 0 0"/>
 			<parent link="${name}_hipassembly"/>
 			<child  link="${name}_upperleg"/>
 			<axis xyz="0 0 1"/>
-			<limit effort="150.0" velocity="12.0"
-				   lower="${-(1+reflect_front)*5*PI/36-(1-reflect_front)*7*PI/36}"
-				   upper="${(1-reflect_front)*5*PI/36+(1+reflect_front)*7*PI/36}"/>
+			<limit effort="${hfe_limit}" velocity="12.0"
+                  lower="${(1-knee_bent_backward)*(hfe_min)*PI/180 + (knee_bent_backward)*(-hfe_max)*PI/180}"
+                  upper="${(1-knee_bent_backward)*(hfe_max)*PI/180 + (knee_bent_backward)*(-hfe_min)*PI/180}"/>
 			<dynamics damping="0.1" friction="0" />
-			<safety_controller k_position="100" k_velocity="100"
-							   soft_lower_limit="${-(1+reflect_front)*5*PI/36-(1-reflect_front)*7*PI/36}"
-							   soft_upper_limit="${(1-reflect_front)*5*PI/36+(1+reflect_front)*7*PI/36}" />
+			<safety_controller k_position="50" k_velocity="10"
+                  lower="${(1-knee_bent_backward)*(hfe_min)*PI/180 + (knee_bent_backward)*(-hfe_max)*PI/180}"
+                  upper="${(1-knee_bent_backward)*(hfe_max)*PI/180 + (knee_bent_backward)*(-hfe_min)*PI/180}"/>
 		</joint>
 		<!-- Lower leg joint -->
 		<joint name="${name}_kfe_joint" type="revolute">
-			<origin xyz="${d_p1p2} 0 0" rpy="0 0 0"/>
+			<origin xyz="${upperleg_length} 0 0" rpy="0 0 0"/>
 			<parent link="${name}_upperleg"/>
 			<child  link="${name}_lowerleg"/>
 			<axis xyz="0 0 1"/>
-			<limit effort="150.0" velocity="12.0"
-				   lower="${-(1+reflect_front)*7*PI/18+(1-reflect_front)*PI/18}"
-				   upper="${(1-reflect_front)*7*PI/18-(1+reflect_front)*PI/18}"/>
+			<limit effort="${kfe_limit}" velocity="12.0"
+                  lower="${(1-knee_bent_backward)*(kfe_min)*PI/180 + (knee_bent_backward)*(-kfe_max)*PI/180}"
+                  upper="${(1-knee_bent_backward)*(kfe_max)*PI/180 + (knee_bent_backward)*(-kfe_min)*PI/180}"/>
 			<dynamics damping="0.1" friction="0" />
-			<safety_controller k_position="100" k_velocity="100"
-							   soft_lower_limit="${-(1+reflect_front)*7*PI/18+(1-reflect_front)*PI/18}"
-							   soft_upper_limit="${(1-reflect_front)*7*PI/18-(1+reflect_front)*PI/18}" />
+			<safety_controller k_position="50" k_velocity="10"
+                  lower="${(1-knee_bent_backward)*(kfe_min)*PI/180 + (knee_bent_backward)*(-kfe_max)*PI/180}"
+                  upper="${(1-knee_bent_backward)*(kfe_max)*PI/180 + (knee_bent_backward)*(-kfe_min)*PI/180}"/>
 		<!-- Foot joint -->
 		</joint>
 		<joint name="${name}_foot_joint" type="fixed">
-			<origin xyz="${d_p2p3} 0 0" rpy="${PI/2} 0 ${-PI/2}"/>
+			<origin xyz="${lowerleg_length} 0 0" rpy="${PI/2} 0 ${-PI/2}"/>
 			<parent link="${name}_lowerleg"/>
 			<child  link="${name}_foot"/>

Commit message: updated trunk mass to include multisense
corrected transform from base to multisense and asus

File: robots/hyq.urdf.xacro (robot description, xacro)
@@ -113,9 +113,9 @@
     <xacro:multisense_sl parent="trunk" prefix="multisense">
 		<!-- <origin xyz="0.741737 0.0191395 0.143229" rpy="-0.0241345 0.446222 -0.0347202"/> -->
-		<origin xyz="0.741737 0.0 0.143229" rpy="-0.0241345 0.446222 -0.0347202"/>
+		<origin xyz="0.761 0.005 0.127" rpy="-0.028 0.515 -0.013"/>
     </xacro:multisense_sl>
 	<!-- Asus Xtion Pro -->
 	<xacro:asus_xtion_camera name="asus" parent="trunk">
-		<origin xyz="0.66489 0.0016545 0.0380496" rpy="0.00740313 0.516618 0.0244919"/>
+		<origin xyz="0.624 -0.013 0.061" rpy="0.018 0.535 0.057"/>
 	</xacro:asus_xtion_camera>
 </robot>

File: urdfs/common.xacro (robot description, xacro)
@@ -21,8 +21,8 @@
 	<!-- Inertial values -->
 	<!-- Trunk with hydraulic system -->
-	<property name="xcom_trunk" value="-0.0004"/>
-	<property name="ycom_trunk" value="-0.0000536"/>
-	<property name="zcom_trunk" value="0.003553"/>
-	<property name="m_trunk" value="59.1"/>
+	<property name="xcom_trunk" value="0.056"/>
+	<property name="ycom_trunk" value="0.0215"/>
+	<property name="zcom_trunk" value="0.00358"/>
+	<property name="m_trunk" value="60.96"/>
 	<property name="ixx_trunk" value="1.5725937"/>
 	<property name="iyy_trunk" value="8.5015928"/>
